File: mcp73123-breakout01.brd (EAGLE design)
At the start: 15.7 x 12.7 mm, 9 parts

Commit message: aesthetic changes
Parts:
- added U$3: OSHW-LOGOS, SparkFun-Aesthetics:OSHW-LOGO-S
- moved BATT 12.7 mm to (13.5, 3.30), turned to 90 degrees
- moved USB/5V 12.5 mm to (2.41, 3.30), turned to 90 degrees
- moved C2 9.55 mm to (10.2, 2.16), turned to 270 degrees
- moved R_STAT 9.22 mm to (10.3, 10.3), turned to 90 degrees
- moved C1 8.38 mm to (7.87, 2.16), turned to 270 degrees
- moved R_PROG 6.41 mm to (7.62, 9.53), turned to 0 degrees
- moved LED_STAT 5.91 mm to (5.21, 4.70), turned to 90 degrees
- moved U$1 2.79 mm to (9.27, 6.35), turned to 0 degrees
- moved U$2 2.79 mm to (7.75, 6.10)
Routing:
- net GND: vias 1 -> 7
Other:
- board text added: "(1.00k)"
- board text added: "CHRG"
- board text added: "Iout: (1.1A)"
- board text added: "Single Cell"
- board text added: "VIN: 4-16V"
- board text removed: "1.00k"
- board text removed: "5V"
- board text removed: "CHARGING"
- board text removed: "Single Cell 1.1 Amp"
