File: mcp73123-breakout01.sch (EAGLE design)
At the start: 9 parts

Commit message: aesthetic changes
Parts:
- added U$3: OSHW-LOGOS, SparkFun-Aesthetics:OSHW-LOGOS
Other:
- note added: "Andrew Duhan 2012"
Changed lines of the file:
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@@
 <part name="R_STAT" library="SparkFun-Passives" deviceset="RESISTOR" device="0603-RES" value="1k"/>
 <part name="U$2" library="myparts" deviceset="DP_LOGO" device=""/>
+<part name="U$3" library="SparkFun-Aesthetics" deviceset="OSHW-LOGO" device="S"/>
 </parts>
 <sheets>
 <sheet>
 <plain>
+<text x="40.64" y="17.78" size="1.778" layer="91">Andrew Duhan 2012</text>
 </plain>
 <instances>
@@
 <instance part="LED_STAT" gate="G$1" x="35.56" y="48.26" rot="R90"/>
 <instance part="R_STAT" gate="G$1" x="45.72" y="48.26" rot="R180"/>
-<instance part="U$2" gate="G$1" x="27.94" y="66.04"/>
+<instance part="U$2" gate="G$1" x="53.34" y="25.4"/>
+<instance part="U$3" gate="G$1" x="25.4" y="25.4"/>
 </instances>
 <busses>
